Commit message: its definitely something

File: models/manipulator.urdf.xacro (robot description, xacro)
@@ -1,5 +1,13 @@
 <?xml version="1.0"?>
-<robot xmlns:xacro="http://ros.org/wiki/xacro" name="simple_arm">
+<robot xmlns:xacro="http://ros.org/wiki/xacro" name="three_link_manipulator">
   <xacro:property name="pi" value="3.141592653589793"/>
+  <!-- Dummy Root Link -->
+  <link name="dummy_root"/>
+  <!-- Fixed joint to base_link -->
+  <joint name="fixed_base" type="fixed">
+    <parent link="dummy_root"/>
+    <child link="base_link"/>
+    <origin xyz="0 0 0" rpy="0 0 0"/>
+  </joint>
   <!-- Base Link -->
   <link name="base_link">
@@ -54,3 +62,68 @@
     </inertial>
   </link>
+  <!-- Joint 2 -->
+  <joint name="joint2" type="revolute">
+    <parent link="link1"/>
+    <child link="link2"/>
+    <origin xyz="0 0 0.5" rpy="0 0 0"/>
+    <axis xyz="0 0 1"/>
+    <limit effort="5" velocity="1" lower="-${pi}" upper="${pi}"/>
+  </joint>
+  <!-- Link 2 -->
+  <link name="link2">
+    <visual>
+      <origin xyz="0 0 0.25" rpy="0 0 0"/>
+      <geometry>
+        <cylinder length="0.5" radius="0.05"/>
+      </geometry>
+      <material name="green">
+        <color rgba="0.2 0.8 0.2 1.0"/>
+      </material>
+    </visual>
+    <collision>
+      <origin xyz="0 0 0.25" rpy="0 0 0"/>
+      <geometry>
+        <cylinder length="0.5" radius="0.05"/>
+      </geometry>
+    </collision>
+    <inertial>
+      <mass value="0.5"/>
+      <inertia ixx="0.005" iyy="0.005" izz="0.005"
+               ixy="0.0" ixz="0.0" iyz="0.0"/>
+    </inertial>
+  </link>
+  <!-- Joint 3 -->
+  <joint name="joint3" type="revolute">
+    <parent link="link2"/>
+    <child link="link3"/>
+    <origin xyz="0 0 0.5" rpy="0 0 0"/>
+    <axis xyz="0 0 1"/>
+    <limit effort="5" velocity="1" lower="-${pi}" upper="${pi}"/>
+  </joint>
+  <!-- Link 3 -->
+  <link name="link3">
+    <visual>
+      <origin xyz="0 0 0.25" rpy="0 0 0"/>
+      <geometry>
+        <cylinder length="0.5" radius="0.05"/>
+      </geometry>
+      <material name="red">
+        <color rgba="0.8 0.2 0.2 1.0"/>
+      </material>
+    </visual>
+    <collision>
+      <origin xyz="0 0 0.25" rpy="0 0 0"/>
+      <geometry>
+        <cylinder length="0.5" radius="0.05"/>
+      </geometry>
+    </collision>
+    <inertial>
+      <mass value="0.5"/>
+      <inertia ixx="0.005" iyy="0.005" izz="0.005"
+               ixy="0.0" ixz="0.0" iyz="0.0"/>
+    </inertial>
+  </link>
+  <gazebo reference="link3">
+    <gravity>false</gravity>
+  </gazebo>
 </robot>

File: urdf/manipulator.urdf (robot description, URDF)
Before this commit: robot simple_arm, 2 links, 1 joints
Links:
- removed link link1
- added link base, mass 0.0
- added link ee_link, mass 0.0; collision box size=0.01 0.01 0.01
- added link forearm_link, mass 3.87; collision mesh filename=file:///home/sam/dev/cpp/arm_ws/src/arm_simulator/meshes/ur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; visual mesh filename=file:///home/sam/dev/cpp/arm_ws/src/arm_simulator/meshes/ur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
- added link shoulder_link, mass 7.778; collision mesh filename=file:///home/sam/dev/cpp/arm_ws/src/arm_simulator/meshes/ur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; visual mesh filename=file:///home/sam/dev/cpp/arm_ws/src/arm_simulator/meshes/ur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
- added link tool0, mass 0.0
- added link upper_arm_link, mass 12.93; collision mesh filename=file:///home/sam/dev/cpp/arm_ws/src/arm_simulator/meshes/ur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; visual mesh filename=file:///home/sam/dev/cpp/arm_ws/src/arm_simulator/meshes/ur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
- added link world
- added link wrist_1_link, mass 1.96; collision mesh filename=file:///home/sam/dev/cpp/arm_ws/src/arm_simulator/meshes/ur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; visual mesh filename=file:///home/sam/dev/cpp/arm_ws/src/arm_simulator/meshes/ur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
- added link wrist_2_link, mass 1.96; collision mesh filename=file:///home/sam/dev/cpp/arm_ws/src/arm_simulator/meshes/ur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; visual mesh filename=file:///home/sam/dev/cpp/arm_ws/src/arm_simulator/meshes/ur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
- added link wrist_3_link, mass 0.202; collision mesh filename=file:///home/sam/dev/cpp/arm_ws/src/arm_simulator/meshes/ur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; visual mesh filename=file:///home/sam/dev/cpp/arm_ws/src/arm_simulator/meshes/ur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
- link base_link: mass 1.0 -> 4.0; geometry collision mesh filename=file:///home/sam/dev/cpp/arm_ws/src/arm_simulator/meshes/ur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; visual mesh filename=file:///home/sam/dev/cpp/arm_ws/src/arm_simulator/meshes/ur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
Joints:
- removed joint joint1
- added joint base_link-base_fixed_joint: type fixed, parent base_link, child base, origin xyz=0 0 0 rpy=0 0 -3.14159265359
- added joint ee_fixed_joint: type fixed, parent wrist_3_link, child ee_link, origin xyz=0.0 0.0922 0.0 rpy=0.0 0.0 1.57079632679
- added joint elbow_joint: type revolute, parent upper_arm_link, child forearm_link, origin xyz=0.0 -0.1719 0.612 rpy=0.0 0.0 0.0, axis 0 1 0, limit lower=-3.14159265359 upper=3.14159265359 effort=150.0 velocity=3.15
- added joint shoulder_lift_joint: type revolute, parent shoulder_link, child upper_arm_link, origin xyz=0.0 0.220941 0.0 rpy=0.0 1.57079632679 0.0, axis 0 1 0, limit lower=-6.28318530718 upper=6.28318530718 effort=330.0 velocity=2.16
- added joint shoulder_pan_joint: type revolute, parent base_link, child shoulder_link, origin xyz=0.0 0.0 0.1273 rpy=0.0 0.0 0.0, axis 0 0 1, limit lower=-6.28318530718 upper=6.28318530718 effort=330.0 velocity=2.16
- added joint world_joint: type fixed, parent world, child base_link, origin xyz=0.0 0.0 0.0 rpy=0.0 0.0 0.0
- added joint wrist_1_joint: type revolute, parent forearm_link, child wrist_1_link, origin xyz=0.0 0.0 0.5723 rpy=0.0 1.57079632679 0.0, axis 0 1 0, limit lower=-6.28318530718 upper=6.28318530718 effort=54.0 velocity=3.2
- added joint wrist_2_joint: type revolute, parent wrist_1_link, child wrist_2_link, origin xyz=0.0 0.1149 0.0 rpy=0.0 0.0 0.0, axis 0 0 1, limit lower=-6.28318530718 upper=6.28318530718 effort=54.0 velocity=3.2
- added joint wrist_3_joint: type revolute, parent wrist_2_link, child wrist_3_link, origin xyz=0.0 0.0 0.1157 rpy=0.0 0.0 0.0, axis 0 1 0, limit lower=-6.28318530718 upper=6.28318530718 effort=54.0 velocity=3.2
- added joint wrist_3_link-tool0_fixed_joint: type fixed, parent wrist_3_link, child tool0, origin xyz=0 0.0922 0 rpy=-1.57079632679 0 0
